File: computer_pcb.kicad_sch (KiCad schematic)
At the start: 59 parts, among them SW1 SW_Push, SW2 SW_Push, SW3 SW_Push

Commit message: added multiplication
Parts:
- added 74HC100, 74HC101, 74HC102, 74HC103, 74HC104, 74HC105, 74HC106, 74HC107, 74HC108, 74HC109, 74HC110, 74HC111, 74HC112, 74HC113, 74HC114, 74HC57, 74HC58, 74HC59, 74HC60, 74HC61, 74HC62, 74HC63, 74HC64, 74HC65, 74HC66, 74HC67, 74HC68, 74HC69, 74HC70, 74HC71, 74HC72, 74HC73, 74HC74, 74HC75, 74HC76, 74HC77, 74HC78, 74HC79, 74HC80, 74HC81, 74HC82, 74HC83, 74HC84, 74HC85, 74HC86, 74HC87, 74HC88, 74HC89, 74HC90, 74HC91, 74HC92, 74HC93, 74HC94, 74HC95, 74HC96, 74HC97, 74HC98, 74HC99: ~, symbol 74xx:74HC00-SSOP-14
- added SW10, SW11, SW4, SW5, SW6, SW7, SW8, SW9: SW_Push, symbol Switch:SW_Push
Connections:
- net +5V: now also 74HC100.14 (VCC), 74HC101.14 (VCC), 74HC102.14 (VCC), 74HC103.14 (VCC), 74HC104.14 (VCC), 74HC105.14 (VCC), 74HC106.14 (VCC), 74HC107.14 (VCC), 74HC108.14 (VCC), 74HC109.14 (VCC), 74HC110.14 (VCC), 74HC111.14 (VCC), 74HC112.14 (VCC), 74HC113.14 (VCC), 74HC114.14 (VCC), 74HC57.14 (VCC), 74HC58.14 (VCC), 74HC59.14 (VCC), 74HC60.14 (VCC), 74HC61.14 (VCC), 74HC62.14 (VCC), 74HC63.14 (VCC), 74HC64.14 (VCC), 74HC65.14 (VCC), 74HC66.14 (VCC), 74HC67.14 (VCC), 74HC68.14 (VCC), 74HC69.14 (VCC), 74HC70.14 (VCC), 74HC71.14 (VCC), 74HC72.14 (VCC), 74HC73.14 (VCC), 74HC74.14 (VCC), 74HC75.14 (VCC), 74HC76.14 (VCC), 74HC77.14 (VCC), 74HC78.14 (VCC), 74HC79.14 (VCC), 74HC80.14 (VCC), 74HC81.14 (VCC), 74HC82.14 (VCC), 74HC83.14 (VCC), 74HC84.14 (VCC), 74HC85.14 (VCC), 74HC86.14 (VCC), 74HC87.14 (VCC), 74HC88.14 (VCC), 74HC89.14 (VCC), 74HC90.14 (VCC), 74HC91.14 (VCC), 74HC92.14 (VCC), 74HC93.14 (VCC), 74HC94.14 (VCC), 74HC95.14 (VCC), 74HC96.14 (VCC), 74HC97.14 (VCC), 74HC98.14 (VCC), 74HC99.14 (VCC), SW10.1, SW11.1, SW4.1, SW5.1, SW6.1, SW7.1, SW8.1, SW9.1
- net GND: now also 74HC100.7 (GND), 74HC101.7 (GND), 74HC102.7 (GND), 74HC103.7 (GND), 74HC104.7 (GND), 74HC105.7 (GND), 74HC106.7 (GND), 74HC107.7 (GND), 74HC108.7 (GND), 74HC109.7 (GND), 74HC110.7 (GND), 74HC111.7 (GND), 74HC112.7 (GND), 74HC113.7 (GND), 74HC114.7 (GND), 74HC57.7 (GND), 74HC58.7 (GND), 74HC59.7 (GND), 74HC60.7 (GND), 74HC61.7 (GND), 74HC62.7 (GND), 74HC63.7 (GND), 74HC64.7 (GND), 74HC65.7 (GND), 74HC66.7 (GND), 74HC67.7 (GND), 74HC68.7 (GND), 74HC69.7 (GND), 74HC70.7 (GND), 74HC71.7 (GND), 74HC72.7 (GND), 74HC73.7 (GND), 74HC74.7 (GND), 74HC75.7 (GND), 74HC76.7 (GND), 74HC77.7 (GND), 74HC78.7 (GND), 74HC79.7 (GND), 74HC80.7 (GND), 74HC81.7 (GND), 74HC82.7 (GND), 74HC83.7 (GND), 74HC84.7 (GND), 74HC85.7 (GND), 74HC86.7 (GND), 74HC87.7 (GND), 74HC88.7 (GND), 74HC89.7 (GND), 74HC90.7 (GND), 74HC91.7 (GND), 74HC92.7 (GND), 74HC93.7 (GND), 74HC94.7 (GND), 74HC95.7 (GND), 74HC96.7 (GND), 74HC97.7 (GND), 74HC98.7 (GND), 74HC99.7 (GND)
- net at 74HC41.10 (3B), 74HC41.2 (1B), 74HC42.1 (1A): now also 74HC58.8 (3Y)
- net at 74HC52.11 (4Y): now also 74HC89.10 (3B), 74HC89.2 (1B), 74HC90.1 (1A)
- net at 74HC40.9 (3A), 74HC47.10 (3B), 74HC47.2 (1B): now also 74HC42.9 (3A), 74HC44.9 (3A), 74HC49.10 (3B), 74HC49.2 (1B), 74HC51.10 (3B), 74HC51.2 (1B), 74HC106.9 (3A), 74HC113.10 (3B), 74HC113.2 (1B), 74HC59.8 (3Y), 74HC60.6 (2Y), 74HC66.8 (3Y)
- net at 74HC47.11 (4Y): now also 74HC83.1 (1A), 74HC83.5 (2B), 74HC84.2 (1B)
- net at 74HC37.10 (3B), 74HC37.2 (1B), 74HC38.1 (1A): now also 74HC59.6 (2Y)
- net at 74HC37.1 (1A), 74HC37.5 (2B), 74HC38.2 (1B): now also 74HC57.8 (3Y)
- net at 74HC43.10 (3B), 74HC43.2 (1B), 74HC44.1 (1A): now also 74HC60.8 (3Y)
- net at 74HC39.10 (3B), 74HC39.2 (1B), 74HC40.1 (1A): now also 74HC58.6 (2Y)
- net at 74HC51.11 (4Y): now also 74HC87.10 (3B), 74HC87.2 (1B), 74HC88.1 (1A)
- net at 74HC49.11 (4Y): now also 74HC85.10 (3B), 74HC85.2 (1B), 74HC86.1 (1A)
- new net: 74HC100.2 (1B), 74HC93.11 (4Y), 74HC99.1 (1A), 74HC99.5 (2B)
- new net: 74HC100.1 (1A), 74HC65.6 (2Y), 74HC99.10 (3B), 74HC99.2 (1B)
- new net: 74HC100.10 (3B), 74HC107.1 (1A), 74HC107.5 (2B), 74HC99.11 (4Y)
- new net: 74HC99.12 (4A), 74HC99.8 (3Y)
- new net: 74HC99.13 (4B), 74HC99.6 (2Y)
- new net: 74HC99.3 (1Y), 74HC99.4 (2A), 74HC99.9 (3A)
- new net: 74HC67.1 (1A), 74HC67.5 (2B), 74HC68.2 (1B)
- new net: 74HC67.10 (3B), 74HC67.2 (1B), 74HC68.1 (1A)
- new net: 74HC67.11 (4Y), 74HC68.10 (3B), 74HC75.1 (1A), 74HC75.5 (2B)
- new net: 74HC67.12 (4A), 74HC67.8 (3Y)
- new net: 74HC67.13 (4B), 74HC67.6 (2Y)
- new net: 74HC67.3 (1Y), 74HC67.4 (2A), 74HC67.9 (3A)
- new net: 74HC59.12 (4A), 74HC59.2 (1B), 74HC60.12 (4A), 74HC60.2 (1B), SW7.2
- new net: 74HC57.13 (4B), 74HC59.13 (4B), 74HC63.13 (4B), 74HC65.13 (4B), SW6.2
- new net: 74HC68.11 (4Y), 74HC76.1 (1A), 74HC76.2 (1B)
- new net: 74HC68.12 (4A), 74HC68.13 (4B), 74HC68.8 (3Y)
- new net: 74HC68.3 (1Y), 74HC68.4 (2A), 74HC68.5 (2B)
- new net: 74HC68.6 (2Y), 74HC76.4 (2A), 74HC76.5 (2B)
- new net: 74HC68.9 (3A), 74HC75.10 (3B), 74HC75.2 (1B)
- new net: 74HC57.1 (1A), 74HC59.1 (1A), 74HC63.1 (1A), 74HC65.1 (1A), SW4.2
- new net: 74HC59.10 (3B), 74HC59.11 (4Y), 74HC59.9 (3A)
- new net: 74HC59.3 (1Y), 74HC59.4 (2A), 74HC59.5 (2B)
- new net: 74HC105.11 (4Y), 74HC106.10 (3B), 74HC113.1 (1A), 74HC113.5 (2B)
- new net: 74HC113.12 (4A), 74HC113.8 (3Y)
- new net: 74HC113.13 (4B), 74HC113.6 (2Y)
- new net: 74HC113.3 (1Y), 74HC113.4 (2A), 74HC113.9 (3A)
- new net: 74HC63.12 (4A), 74HC63.2 (1B), 74HC64.12 (4A), 74HC64.2 (1B), SW9.2
- new net: 74HC100.11 (4Y), 74HC108.1 (1A), 74HC108.2 (1B)
- new net: 74HC101.1 (1A), 74HC101.5 (2B), 74HC102.2 (1B), 74HC108.11 (4Y)
- new net: 74HC108.12 (4A), 74HC108.6 (2Y)
- new net: 74HC108.13 (4B), 74HC108.3 (1Y)
- new net: 74HC100.6 (2Y), 74HC108.4 (2A), 74HC108.5 (2B)
- new net: 74HC63.10 (3B), 74HC63.11 (4Y), 74HC63.9 (3A)
- new net: 74HC63.3 (1Y), 74HC63.4 (2A), 74HC63.5 (2B)
- new net: 74HC63.6 (2Y), 74HC83.10 (3B), 74HC83.2 (1B), 74HC84.1 (1A)
- new net: 74HC63.8 (3Y), 74HC86.9 (3A), 74HC93.10 (3B), 74HC93.2 (1B)
- new net: 74HC74.11 (4Y), 74HC82.1 (1A), 74HC82.2 (1B)
- new net: 74HC82.12 (4A), 74HC82.6 (2Y)
- new net: 74HC82.13 (4B), 74HC82.3 (1Y)
- new net: 74HC74.6 (2Y), 74HC82.4 (2A), 74HC82.5 (2B)
- new net: 74HC105.1 (1A), 74HC105.5 (2B), 74HC106.2 (1B), 74HC112.11 (4Y)
- new net: 74HC105.10 (3B), 74HC105.2 (1B), 74HC106.1 (1A), 74HC98.11 (4Y)
- new net: 74HC105.12 (4A), 74HC105.8 (3Y)
- new net: 74HC105.13 (4B), 74HC105.6 (2Y)
- new net: 74HC105.3 (1Y), 74HC105.4 (2A), 74HC105.9 (3A)
- new net: 74HC58.1 (1A), 74HC60.1 (1A), 74HC64.1 (1A), 74HC66.1 (1A), SW8.2
- new net: 74HC83.11 (4Y), 74HC84.10 (3B), 74HC91.1 (1A), 74HC91.5 (2B)
- new net: 74HC84.9 (3A), 74HC91.10 (3B), 74HC91.2 (1B)
- new net: 74HC91.12 (4A), 74HC91.8 (3Y)
- new net: 74HC91.13 (4B), 74HC91.6 (2Y)
- new net: 74HC91.3 (1Y), 74HC91.4 (2A), 74HC91.9 (3A)
- new net: 74HC103.1 (1A), 74HC103.5 (2B), 74HC104.2 (1B), 74HC110.11 (4Y)
- new net: 74HC103.10 (3B), 74HC103.2 (1B), 74HC104.1 (1A), 74HC97.11 (4Y)
- new net: 74HC103.11 (4Y), 74HC104.10 (3B), 74HC111.1 (1A), 74HC111.5 (2B)
- new net: 74HC103.12 (4A), 74HC103.8 (3Y)
- new net: 74HC103.13 (4B), 74HC103.6 (2Y)
- new net: 74HC103.3 (1Y), 74HC103.4 (2A), 74HC103.9 (3A)
- new net: 74HC87.1 (1A), 74HC87.5 (2B), 74HC88.2 (1B), 74HC94.11 (4Y)
- new net: 74HC87.11 (4Y), 74HC88.10 (3B), 74HC95.1 (1A), 74HC95.5 (2B)
- new net: 74HC87.12 (4A), 74HC87.8 (3Y)
- new net: 74HC87.13 (4B), 74HC87.6 (2Y)
- new net: 74HC87.3 (1Y), 74HC87.4 (2A), 74HC87.9 (3A)
- new net: 74HC84.11 (4Y), 74HC92.1 (1A), 74HC92.2 (1B)
- new net: 74HC84.12 (4A), 74HC84.13 (4B), 74HC84.8 (3Y)
- new net: 74HC84.3 (1Y), 74HC84.4 (2A), 74HC84.5 (2B)
- new net: 74HC84.6 (2Y), 74HC92.4 (2A), 74HC92.5 (2B)
- new net: 74HC73.1 (1A), 74HC73.5 (2B), 74HC74.2 (1B), 74HC80.11 (4Y)
- new net: 74HC73.10 (3B), 74HC73.2 (1B), 74HC74.1 (1A)
- new net: 74HC73.11 (4Y), 74HC74.10 (3B), 74HC81.1 (1A), 74HC81.5 (2B)
- new net: 74HC73.12 (4A), 74HC73.8 (3Y)
- new net: 74HC73.13 (4B), 74HC73.6 (2Y)
- new net: 74HC73.3 (1Y), 74HC73.4 (2A), 74HC73.9 (3A)
- new net: 74HC57.12 (4A), 74HC57.2 (1B), 74HC58.12 (4A), 74HC58.2 (1B), SW5.2
- new net: 74HC64.6 (2Y), 74HC88.9 (3A), 74HC95.10 (3B), 74HC95.2 (1B)
- new net: 74HC101.10 (3B), 74HC101.2 (1B), 74HC102.1 (1A), 74HC95.11 (4Y)
- new net: 74HC95.12 (4A), 74HC95.8 (3Y)
- new net: 74HC95.13 (4B), 74HC95.6 (2Y)
- new net: 74HC95.3 (1Y), 74HC95.4 (2A), 74HC95.9 (3A)
- new net: 74HC65.12 (4A), 74HC65.2 (1B), 74HC66.12 (4A), 74HC66.2 (1B), SW11.2
- new net: 74HC58.10 (3B), 74HC58.11 (4Y), 74HC58.9 (3A)
- new net: 74HC58.13 (4B), 74HC60.13 (4B), 74HC64.13 (4B), 74HC66.13 (4B), SW10.2
- new net: 74HC58.3 (1Y), 74HC58.4 (2A), 74HC58.5 (2B)
- new net: 74HC89.11 (4Y), 74HC90.10 (3B), 74HC97.1 (1A), 74HC97.5 (2B)
- new net: 74HC90.11 (4Y), 74HC98.1 (1A), 74HC98.2 (1B)
- new net: 74HC90.12 (4A), 74HC90.13 (4B), 74HC90.8 (3Y)
- new net: 74HC89.1 (1A), 74HC89.5 (2B), 74HC90.2 (1B), 74HC96.11 (4Y)
- new net: 74HC90.3 (1Y), 74HC90.4 (2A), 74HC90.5 (2B)
- new net: 74HC90.6 (2Y), 74HC98.4 (2A), 74HC98.5 (2B)
- new net: 74HC64.8 (3Y), 74HC90.9 (3A), 74HC97.10 (3B), 74HC97.2 (1B)
- new net: 74HC104.11 (4Y), 74HC112.1 (1A), 74HC112.2 (1B)
- new net: 74HC104.12 (4A), 74HC104.13 (4B), 74HC104.8 (3Y)
- new net: 74HC104.3 (1Y), 74HC104.4 (2A), 74HC104.5 (2B)
- new net: 74HC104.6 (2Y), 74HC112.4 (2A), 74HC112.5 (2B)
- new net: 74HC104.9 (3A), 74HC111.10 (3B), 74HC111.2 (1B), 74HC66.6 (2Y)
- new net: 74HC69.10 (3B), 74HC69.2 (1B), 74HC70.1 (1A)
- new net: 74HC69.11 (4Y), 74HC70.10 (3B), 74HC77.1 (1A), 74HC77.5 (2B)
- new net: 74HC70.11 (4Y), 74HC78.1 (1A), 74HC78.2 (1B)
- new net: 74HC70.12 (4A), 74HC70.13 (4B), 74HC70.8 (3Y)
- new net: 74HC69.1 (1A), 74HC69.5 (2B), 74HC70.2 (1B), 74HC76.11 (4Y)
- new net: 74HC70.3 (1Y), 74HC70.4 (2A), 74HC70.5 (2B)
- new net: 74HC70.6 (2Y), 74HC78.4 (2A), 74HC78.5 (2B)
- new net: 74HC70.9 (3A), 74HC77.10 (3B), 74HC77.2 (1B)
- new net: 74HC71.1 (1A), 74HC71.5 (2B), 74HC72.2 (1B), 74HC78.11 (4Y)
- new net: 74HC78.12 (4A), 74HC78.6 (2Y)
- new net: 74HC78.13 (4B), 74HC78.3 (1Y)
- new net: 74HC83.12 (4A), 74HC83.8 (3Y)
- new net: 74HC83.13 (4B), 74HC83.6 (2Y)
- new net: 74HC83.3 (1Y), 74HC83.4 (2A), 74HC83.9 (3A)
- new net: 74HC101.11 (4Y), 74HC102.10 (3B), 74HC109.1 (1A), 74HC109.5 (2B)
- new net: 74HC102.11 (4Y), 74HC110.1 (1A), 74HC110.2 (1B)
- new net: 74HC102.12 (4A), 74HC102.13 (4B), 74HC102.8 (3Y)
- new net: 74HC102.3 (1Y), 74HC102.4 (2A), 74HC102.5 (2B)
- new net: 74HC102.6 (2Y), 74HC110.4 (2A), 74HC110.5 (2B)
- new net: 74HC102.9 (3A), 74HC109.10 (3B), 74HC109.2 (1B), 74HC65.8 (3Y)
- new net: 74HC77.12 (4A), 74HC77.8 (3Y)
- new net: 74HC77.13 (4B), 74HC77.6 (2Y)
- new net: 74HC77.3 (1Y), 74HC77.4 (2A), 74HC77.9 (3A)
- new net: 74HC110.12 (4A), 74HC110.6 (2Y)
- new net: 74HC110.13 (4B), 74HC110.3 (1Y)
- new net: 74HC86.11 (4Y), 74HC94.1 (1A), 74HC94.2 (1B)
- new net: 74HC94.12 (4A), 74HC94.6 (2Y)
- new net: 74HC94.13 (4B), 74HC94.3 (1Y)
- new net: 74HC86.6 (2Y), 74HC94.4 (2A), 74HC94.5 (2B)
- new net: 74HC65.10 (3B), 74HC65.11 (4Y), 74HC65.9 (3A)
- new net: 74HC65.3 (1Y), 74HC65.4 (2A), 74HC65.5 (2B)
- new net: 74HC98.12 (4A), 74HC98.6 (2Y)
- new net: 74HC98.13 (4B), 74HC98.3 (1Y)
- new net: 74HC57.10 (3B), 74HC57.11 (4Y), 74HC57.9 (3A)
- new net: 74HC57.3 (1Y), 74HC57.4 (2A), 74HC57.5 (2B)
- new net: 74HC85.11 (4Y), 74HC86.10 (3B), 74HC93.1 (1A), 74HC93.5 (2B)
- new net: 74HC86.12 (4A), 74HC86.13 (4B), 74HC86.8 (3Y)
- new net: 74HC85.1 (1A), 74HC85.5 (2B), 74HC86.2 (1B), 74HC92.11 (4Y)
- new net: 74HC86.3 (1Y), 74HC86.4 (2A), 74HC86.5 (2B)
- new net: 74HC74.9 (3A), 74HC81.10 (3B), 74HC81.2 (1B)
- new net: 74HC81.12 (4A), 74HC81.8 (3Y)
- new net: 74HC81.13 (4B), 74HC81.6 (2Y)
- new net: 74HC81.3 (1Y), 74HC81.4 (2A), 74HC81.9 (3A)
- new net: 74HC100.12 (4A), 74HC100.13 (4B), 74HC100.8 (3Y)
- new net: 74HC100.3 (1Y), 74HC100.4 (2A), 74HC100.5 (2B)
- new net: 74HC100.9 (3A), 74HC107.10 (3B), 74HC107.2 (1B)
- new net: 74HC71.10 (3B), 74HC71.2 (1B), 74HC72.1 (1A)
- new net: 74HC71.11 (4Y), 74HC72.10 (3B), 74HC79.1 (1A), 74HC79.5 (2B)
- new net: 74HC72.11 (4Y), 74HC80.1 (1A), 74HC80.2 (1B)
- new net: 74HC72.12 (4A), 74HC72.13 (4B), 74HC72.8 (3Y)
- new net: 74HC72.3 (1Y), 74HC72.4 (2A), 74HC72.5 (2B)
- new net: 74HC72.6 (2Y), 74HC80.4 (2A), 74HC80.5 (2B)
- new net: 74HC72.9 (3A), 74HC79.10 (3B), 74HC79.2 (1B)
- new net: 74HC80.12 (4A), 74HC80.6 (2Y)
- new net: 74HC80.13 (4B), 74HC80.3 (1Y)
- new net: 74HC85.12 (4A), 74HC85.8 (3Y)
- new net: 74HC85.13 (4B), 74HC85.6 (2Y)
- new net: 74HC85.3 (1Y), 74HC85.4 (2A), 74HC85.9 (3A)
- new net: 74HC74.12 (4A), 74HC74.13 (4B), 74HC74.8 (3Y)
- new net: 74HC74.3 (1Y), 74HC74.4 (2A), 74HC74.5 (2B)
- new net: 74HC92.12 (4A), 74HC92.6 (2Y)
- new net: 74HC92.13 (4B), 74HC92.3 (1Y)
- new net: 74HC101.12 (4A), 74HC101.8 (3Y)
- new net: 74HC101.13 (4B), 74HC101.6 (2Y)
- new net: 74HC101.3 (1Y), 74HC101.4 (2A), 74HC101.9 (3A)
- new net: 74HC76.12 (4A), 74HC76.6 (2Y)
- new net: 74HC76.13 (4B), 74HC76.3 (1Y)
- new net: 74HC69.12 (4A), 74HC69.8 (3Y)
- new net: 74HC69.13 (4B), 74HC69.6 (2Y)
- new net: 74HC69.3 (1Y), 74HC69.4 (2A), 74HC69.9 (3A)
- new net: 74HC60.10 (3B), 74HC60.11 (4Y), 74HC60.9 (3A)
- new net: 74HC60.3 (1Y), 74HC60.4 (2A), 74HC60.5 (2B)
- new net: 74HC106.11 (4Y), 74HC114.1 (1A), 74HC114.2 (1B)
- new net: 74HC106.12 (4A), 74HC106.13 (4B), 74HC106.8 (3Y)
- new net: 74HC106.3 (1Y), 74HC106.4 (2A), 74HC106.5 (2B)
- new net: 74HC106.6 (2Y), 74HC114.4 (2A), 74HC114.5 (2B)
- new net: 74HC75.12 (4A), 74HC75.8 (3Y)
- new net: 74HC75.13 (4B), 74HC75.6 (2Y)
- new net: 74HC75.3 (1Y), 74HC75.4 (2A), 74HC75.9 (3A)
- new net: 74HC64.10 (3B), 74HC64.11 (4Y), 74HC64.9 (3A)
- new net: 74HC64.3 (1Y), 74HC64.4 (2A), 74HC64.5 (2B)
- new net: 74HC89.12 (4A), 74HC89.8 (3Y)
- new net: 74HC89.13 (4B), 74HC89.6 (2Y)
- new net: 74HC89.3 (1Y), 74HC89.4 (2A), 74HC89.9 (3A)
- new net: 74HC114.12 (4A), 74HC114.6 (2Y)
- new net: 74HC114.13 (4B), 74HC114.3 (1Y)
- new net: 74HC111.12 (4A), 74HC111.8 (3Y)
- new net: 74HC111.13 (4B), 74HC111.6 (2Y)
- new net: 74HC111.3 (1Y), 74HC111.4 (2A), 74HC111.9 (3A)
- new net: 74HC79.12 (4A), 74HC79.8 (3Y)
- new net: 74HC79.13 (4B), 74HC79.6 (2Y)
- new net: 74HC79.3 (1Y), 74HC79.4 (2A), 74HC79.9 (3A)
- new net: 74HC112.12 (4A), 74HC112.6 (2Y)
- new net: 74HC112.13 (4B), 74HC112.3 (1Y)
- new net: 74HC66.10 (3B), 74HC66.11 (4Y), 74HC66.9 (3A)
- new net: 74HC66.3 (1Y), 74HC66.4 (2A), 74HC66.5 (2B)
- new net: 74HC88.11 (4Y), 74HC96.1 (1A), 74HC96.2 (1B)
- new net: 74HC96.12 (4A), 74HC96.6 (2Y)
- new net: 74HC96.13 (4B), 74HC96.3 (1Y)
- new net: 74HC88.6 (2Y), 74HC96.4 (2A), 74HC96.5 (2B)
- new net: 74HC107.12 (4A), 74HC107.8 (3Y)
- new net: 74HC107.13 (4B), 74HC107.6 (2Y)
- new net: 74HC107.3 (1Y), 74HC107.4 (2A), 74HC107.9 (3A)
- new net: 74HC93.12 (4A), 74HC93.8 (3Y)
- new net: 74HC93.13 (4B), 74HC93.6 (2Y)
- new net: 74HC93.3 (1Y), 74HC93.4 (2A), 74HC93.9 (3A)
- new net: 74HC109.12 (4A), 74HC109.8 (3Y)
- new net: 74HC109.13 (4B), 74HC109.6 (2Y)
- new net: 74HC109.3 (1Y), 74HC109.4 (2A), 74HC109.9 (3A)
- new net: 74HC97.12 (4A), 74HC97.8 (3Y)
- new net: 74HC97.13 (4B), 74HC97.6 (2Y)
- new net: 74HC97.3 (1Y), 74HC97.4 (2A), 74HC97.9 (3A)
- new net: 74HC71.12 (4A), 74HC71.8 (3Y)
- new net: 74HC71.13 (4B), 74HC71.6 (2Y)
- new net: 74HC71.3 (1Y), 74HC71.4 (2A), 74HC71.9 (3A)
- new net: 74HC88.12 (4A), 74HC88.13 (4B), 74HC88.8 (3Y)
- new net: 74HC88.3 (1Y), 74HC88.4 (2A), 74HC88.5 (2B)
Other:
- moved on the sheet: SW1, SW2, SW3

Commit message: assigned footprint
Parts:
- removed 74HC53, 74HC54, 74HC55, 74HC56, 74HC61, 74HC62: ~, symbol 74xx:74HC00-SSOP-14
- 74HC1, 74HC10, 74HC100, 74HC101, 74HC102, 74HC103, 74HC104, 74HC105, 74HC106, 74HC107, 74HC108, 74HC109, 74HC11, 74HC110, 74HC111, 74HC112, 74HC113, 74HC114, 74HC12, 74HC13, 74HC14, 74HC15, 74HC16, 74HC17, 74HC18, 74HC19, 74HC2, 74HC20, 74HC21, 74HC22, 74HC23, 74HC24, 74HC25, 74HC26, 74HC27, 74HC28, 74HC29, 74HC3, 74HC30, 74HC31, 74HC32, 74HC33, 74HC34, 74HC35, 74HC36, 74HC37, 74HC38, 74HC39, 74HC4, 74HC40, 74HC41, 74HC42, 74HC43, 74HC44, 74HC45, 74HC46, 74HC47, 74HC48, 74HC49, 74HC5, 74HC50, 74HC51, 74HC52, 74HC57, 74HC58, 74HC59, 74HC6, 74HC60, 74HC63, 74HC64, 74HC65, 74HC66, 74HC67, 74HC68, 74HC69, 74HC7, 74HC70, 74HC71, 74HC72, 74HC73, 74HC74, 74HC75, 74HC76, 74HC77, 74HC78, 74HC79, 74HC8, 74HC80, 74HC81, 74HC82, 74HC83, 74HC84, 74HC85, 74HC86, 74HC87, 74HC88, 74HC89, 74HC9, 74HC90, 74HC91, 74HC92, 74HC93, 74HC94, 74HC95, 74HC96, 74HC97, 74HC98, 74HC99: footprint (none) -> Package_SO:SSOP-14_5.3x6.2mm_P0.65mm
- SW1, SW10, SW11, SW2, SW3, SW4, SW5, SW6, SW7, SW8, SW9: footprint (none) -> Button_Switch_Keyboard:SW_Cherry_MX_1.00u_PCB
